Commit message: ur_description: changed ur10 xacro model

File: ur_description/urdf/ur10.urdf.xacro (robot description, xacro)
@@ -49,8 +49,8 @@
     </visual>
     <collision>
-      <geometry>
-        <mesh filename="package://ur_description/meshes/ur10/collision/Base.stl" />
-      </geometry>
-      <origin xyz="0.0 0.0 0.003" rpy="0.0 0.0 ${3.0 * pi / 4.0}" />
+      <origin rpy="0 0 0" xyz="0 0 0.025"/>
+      <geometry>
+        <cylinder length="0.04" radius="0.09"/>
+      </geometry>
     </collision>
     <inertial>
@@ -64,5 +64,5 @@
     <origin xyz="0.0 0.0 ${shoulder_height}" rpy="0.0 0.0 0.0" />
     <axis xyz="0.0 0.0 1.0" />
-    <limit lower="${-2.0 * pi}" upper="${2.0 * pi}" effort="330.0" velocity="2.16"/>
+    <limit lower="${-pi/2.0}" upper="${3.0 * pi / 2.0}" effort="330.0" velocity="2.16"/>
     <dynamics damping="1.2" friction="0.0"/>
   </joint>
@@ -75,7 +75,8 @@
     </visual>
     <collision>
-      <geometry>
-        <mesh filename="package://ur_description/meshes/ur10/collision/Shoulder.stl" />
-      </geometry>
+		<origin rpy="0 0 0" xyz="0 0 0"/>
+		<geometry>
+			<cylinder length="0.17" radius="0.08"/>
+		</geometry>
     </collision>
     <inertial>
@@ -90,5 +91,5 @@
     <origin xyz="0.0 ${shoulder_offset} 0.0" rpy="0.0 ${pi / 2.0} 0.0" />
     <axis xyz="0.0 1.0 0.0" />
-    <limit lower="${-2.0 * pi}" upper="${2.0 * pi}" effort="10.0" velocity="${pi}"/>
+    <limit lower="${-pi}" upper="${pi}" effort="10.0" velocity="${pi}"/>
     <dynamics damping="1.2" friction="0.0"/>
   </joint>
@@ -101,10 +102,11 @@
       <material name="UR/Blue" />
     </visual>
-    <collision>
-      <geometry>
-        <mesh filename="package://ur_description/meshes/ur10/collision/UpperArm.stl" />
-      </geometry>
-       <origin xyz="0.0 0.0 0.0" rpy="0.0 0.0 0.0" />
-    </collision>
+	<collision>
+		<origin rpy="0 0 0" xyz="0 0 0.30"/>
+		<geometry>
+			<cylinder length="0.7" radius="0.05"/>
+		</geometry>
+		<origin rpy="0.0 0.0 0.0" xyz="0.0 0.0 0.0"/>
+	</collision>
     <inertial>
       <mass value="${upper_arm_mass}" />
@@ -118,5 +120,5 @@
     <origin xyz="0.0 ${-elbow_offset} ${upper_arm_length}" rpy="0.0 0.0 0.0" />
     <axis xyz="0.0 1.0 0.0" />
-    <limit lower="${-2.0 * pi}" upper="${2.0 * pi}" effort="150.0" velocity="${pi}"/>
+    <limit lower="${-pi}" upper="${pi}" effort="150.0" velocity="${pi}"/>
     <dynamics damping="0.6" friction="0.0"/>
   </joint>
@@ -128,9 +130,10 @@
       <material name="UR/Grey" />
     </visual>
-    <collision>
-      <geometry>
-        <mesh filename="package://ur_description/meshes/ur10/collision/Forearm.stl" />
-      </geometry>
-    </collision>
+	<collision>
+		<origin rpy="0 0 0" xyz="0 0 0.28"/>
+ 		<geometry>
+			<cylinder length="0.675" radius="0.04"/>
+		</geometry>
+	</collision>
     <inertial>
       <mass value="${forearm_mass}" />
@@ -144,5 +147,5 @@
     <origin xyz="0.0 0.0 ${forearm_length}" rpy="0.0 ${pi / 2.0} 0.0" />
     <axis xyz="0.0 1.0 0.0" />
-    <limit lower="${-2.0 * pi}" upper="${2.0 * pi}" effort="54.0" velocity="${pi}"/>
+    <limit lower="${-pi}" upper="${pi}" effort="54.0" velocity="${pi}"/>
     <dynamics damping="0.6" friction="0.0"/>
   </joint>
@@ -156,8 +159,8 @@
     </visual>
     <collision>
-      <geometry>
-        <mesh filename="package://ur_description/meshes/ur10/collision/Wrist1.stl" />
-      </geometry>
-      <origin xyz="0.0 ${wrist_1_length} 0.0" rpy="0.0 0 0.0" />
+    	<origin rpy="0 0 0" xyz="0.0 0.113 0.002"/>
+      	<geometry>
+        	<cylinder length="0.116" radius="0.045"/>
+      	</geometry>
     </collision>
     <inertial>
@@ -167,10 +170,10 @@
     </inertial>
   </link>
-    <joint name="${prefix}wrist_2_joint" type="revolute">
+  <joint name="${prefix}wrist_2_joint" type="revolute">
     <parent link="${prefix}wrist_1_link" />
     <child link = "${prefix}wrist_2_link" />
     <origin xyz="0.0 ${wrist_1_length} 0.0" rpy="0.0 0.0 0.0" />
     <axis xyz="0.0 0.0 1.0" />
-    <limit lower="${-2.0 * pi}" upper="${2.0 * pi}" effort="54.0" velocity="${pi}"/>
+    <limit lower="${-pi}" upper="${pi}" effort="54.0" velocity="${pi}"/>
     <dynamics damping="0.6" friction="0.0"/>
   </joint>
@@ -184,8 +187,8 @@
     </visual>
     <collision>
-      <geometry>
-        <mesh filename="package://ur_description/meshes/ur10/collision/Wrist2.stl" />
-      </geometry>
-      <origin xyz="0.0 0.0 ${wrist_2_length}" rpy="0.0 0.0 0.0" />
+      <origin rpy="${pi/2.0} 0 0" xyz="0.0 0 0.11"/>
+      <geometry>
+        <cylinder length="0.11" radius="0.045"/>
+      </geometry>
     </collision>
     <inertial>
@@ -200,5 +203,5 @@
     <origin xyz="0.0 0.0 ${wrist_2_length}" rpy="0.0 0.0 0.0" />
     <axis xyz="0.0 1.0 0.0" />
-    <limit lower="${-2.0 * pi}" upper="${2.0 * pi}" effort="54.0" velocity="${pi}"/>
+    <limit lower="${-pi}" upper="${pi}" effort="54.0" velocity="${pi}"/>
     <dynamics damping="0.6" friction="0.0"/>
   </joint>
@@ -212,8 +215,8 @@
     </visual>
     <collision>
-      <geometry>
-        <mesh filename="package://ur_description/meshes/ur10/collision/Wrist3.stl" />
-      </geometry>
-      <origin xyz="0.0 ${wrist_3_length} 0.0" rpy="0.0 0.0 0" />
+      <origin rpy="${pi/2.0} 0 0" xyz="0 0.068 0"/>
+      <geometry>
+        <cylinder length="0.02" radius="0.045"/>
+      </geometry>
     </collision>
     <inertial>

Commit message: ur_description: larger radius of wrist collision models due to attached cables ur_driver: server fix, is set to aborted when target is not reached

File: ur_description/urdf/ur10.urdf.xacro (robot description, xacro)
@@ -161,5 +161,5 @@
     	<origin rpy="0 0 0" xyz="0.0 0.113 0.002"/>
       	<geometry>
-        	<cylinder length="0.116" radius="0.045"/>
+        	<cylinder length="0.116" radius="0.055"/>
       	</geometry>
     </collision>
@@ -189,5 +189,5 @@
       <origin rpy="${pi/2.0} 0 0" xyz="0.0 0 0.11"/>
       <geometry>
-        <cylinder length="0.11" radius="0.045"/>
+        <cylinder length="0.11" radius="0.055"/>
       </geometry>
     </collision>
@@ -217,5 +217,5 @@
       <origin rpy="${pi/2.0} 0 0" xyz="0 0.068 0"/>
       <geometry>
-        <cylinder length="0.02" radius="0.045"/>
+        <cylinder length="0.02" radius="0.055"/>
       </geometry>
     </collision>

Commit message: New robot collision model

File: ur_description/urdf/ur10.urdf.xacro (robot description, xacro)
@@ -80,4 +80,10 @@
 		</geometry>
     </collision>
+    <collision>
+      <origin rpy="0 ${pi/2.0} ${pi/2}" xyz="0 0.1 0"/>
+		  <geometry>
+			  <cylinder length="0.28" radius="0.08"/>
+		  </geometry>
+    </collision>
     <inertial>
       <mass value="${shoulder_mass}" />
@@ -136,4 +142,10 @@
 		</geometry>
 	</collision>
+  <collision>
+      <origin rpy="0 ${pi/2.0} ${pi/2}" xyz="0 0.07 0"/>
+		  <geometry>
+			  <cylinder length="0.24" radius="0.07"/>
+		  </geometry>
+    </collision>
     <inertial>
       <mass value="${forearm_mass}" />
@@ -192,4 +204,10 @@
       </geometry>
     </collision>
+    <collision>
+      <origin rpy="0 ${pi/2.0} ${pi/2}" xyz="0 -0.05 0"/>
+		  <geometry>
+			  <cylinder length="0.22" radius="0.05"/>
+		  </geometry>
+    </collision>
     <inertial>
       <mass value="${wrist_2_mass}" />

Commit message: reverse collision radius changes

File: ur_description/urdf/ur10.urdf.xacro (robot description, xacro)
@@ -161,5 +161,5 @@
     	<origin rpy="0 0 0" xyz="0.0 0.113 0.002"/>
       	<geometry>
-        	<cylinder length="0.116" radius="0.055"/>
+        	<cylinder length="0.116" radius="0.045"/>
       	</geometry>
     </collision>
@@ -189,5 +189,5 @@
       <origin rpy="${pi/2.0} 0 0" xyz="0.0 0 0.11"/>
       <geometry>
-        <cylinder length="0.11" radius="0.055"/>
+        <cylinder length="0.11" radius="0.045"/>
       </geometry>
     </collision>
@@ -217,5 +217,5 @@
       <origin rpy="${pi/2.0} 0 0" xyz="0 0.068 0"/>
       <geometry>
-        <cylinder length="0.02" radius="0.055"/>
+        <cylinder length="0.02" radius="0.045"/>
       </geometry>
     </collision>

Commit message: collision fix and tolerance attempt to fix :)

File: ur_description/urdf/ur10.urdf.xacro (robot description, xacro)
@@ -176,4 +176,10 @@
       	</geometry>
     </collision>
+    <collision>
+      <origin rpy="0 ${pi/2.0} ${pi/2}" xyz="0 0.07 0"/>
+      <geometry>
+      	<cylinder length="0.09" radius="0.05"/>
+      </geometry>
+    </collision>
     <inertial>
       <mass value="${wrist_1_mass}" />
@@ -204,4 +210,5 @@
       </geometry>
     </collision>
+  <!--
     <collision>
       <origin rpy="0 ${pi/2.0} ${pi/2}" xyz="0 -0.05 0"/>
@@ -210,4 +217,5 @@
 		  </geometry>
     </collision>
+-->
     <inertial>
       <mass value="${wrist_2_mass}" />
@@ -221,5 +229,5 @@
     <origin xyz="0.0 0.0 ${wrist_2_length}" rpy="0.0 0.0 0.0" />
     <axis xyz="0.0 1.0 0.0" />
-    <limit lower="${-pi}" upper="${pi}" effort="54.0" velocity="${pi}"/>
+    <limit lower="${-pi + (pi/4.0)}" upper="${pi + (pi/4.0)}" effort="54.0" velocity="${pi}"/>
     <dynamics damping="0.6" friction="0.0"/>
   </joint>

Commit message: collision fix and server set to succeeded info msg

File: ur_description/urdf/ur10.urdf.xacro (robot description, xacro)
@@ -139,5 +139,5 @@
 		<origin rpy="0 0 0" xyz="0 0 0.28"/>
  		<geometry>
-			<cylinder length="0.675" radius="0.04"/>
+			<cylinder length="0.635" radius="0.04"/>
 		</geometry>
 	</collision>
@@ -177,7 +177,7 @@
     </collision>
     <collision>
-      <origin rpy="0 ${pi/2.0} ${pi/2}" xyz="0 0.07 0"/>
-      <geometry>
-      	<cylinder length="0.09" radius="0.05"/>
+      <origin rpy="0 ${pi/2.0} ${pi/2}" xyz="0.0 0.06 0"/>
+      <geometry>
+      	<cylinder length="0.09" radius="0.045"/>
       </geometry>
     </collision>
